Commit message: Add the V1-forearm mount adapter, Blender URDF/USD pipeline, and measurement docs
- measure the elbow_roll flange (D10 hub, 6xM3 on BCD36) and the V1 cuff
  (OD84/ID70) from the repo's own meshes; design the printable adapter
  (STL + STEP + drawing + print guide) and fix mount.right at z = 0.012
- teach generate_urdf.py to hang the adapter on the arm_*_mount links
  (visual/collision/inertial, inverse-mount origin) and regenerate the URDFs
- add scripts/blender_import_urdf.py (URDF -> live empty tree in Blender)
  and scripts/blender_export_usd.py (flat visual USD + UsdPhysics
  articulation: 81 bodies, 48 revolute / 33 fixed joints, convex-hull
  collisions); track *.usdc and *.blend with LFS, binaries follow separately
- document the finger-coupling measurement procedure and today's work log

Co-Authored-By: Claude Fable 5 <noreply@anthropic.com>
Claude-Session: https://claude.ai/code/session_016EB6FLo38RgDjgCtRSd4wo

File: ros2_ws/src/berkeley_humanoid_lite_description/urdf/berkeley_humanoid_lite_dexhand.urdf (robot description, URDF)
Before this commit: robot berkeley-humanoid-lite, 42 links, 41 joints
Links:
- link arm_right_mount: mass None -> 0.0508; geometry collision mesh filename=package://berkeley_humanoid_lite_description/meshes_adapter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 scale=0.001 0.001 0.001; visual mesh filename=package://berkeley_humanoid_lite_description/meshes_adapter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 scale=0.001 0.001 0.001
Joints:
- joint arm_right_forearm_mount: origin xyz=0 0 0 rpy=0 0 0 -> xyz=0 0 0.012 rpy=0 0 0

File: ros2_ws/src/berkeley_humanoid_lite_description/urdf/berkeley_humanoid_lite_tuning.urdf (robot description, URDF)
Before this commit: robot berkeley-humanoid-lite, 87 links, 86 joints
Links:
- link arm_left_mount: mass None -> 0.0508; geometry collision mesh filename=package://berkeley_humanoid_lite_description/meshes_adapter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 scale=0.001 0.001 0.001; visual mesh filename=package://berkeley_humanoid_lite_description/meshes_adapter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 scale=0.001 0.001 0.001
- link arm_right_elbow_roll: geometry collision cylinder length=0.12 radius=0.03; visual mesh filename=package://berkeley_humanoid_lite_description/meshes/arm_rig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
Joints:
- joint arm_left_forearm_mount: origin xyz=0 -0 0 rpy=-0 0 -0 -> xyz=0 -0 0.012 rpy=-0 0 -0

File: ros2_ws/src/berkeley_humanoid_lite_description/urdf/berkeley_humanoid_lite_v1arm.urdf (robot description, URDF)
Before this commit: robot berkeley-humanoid-lite, 82 links, 81 joints
Links:
- link arm_left_mount: mass None -> 0.0508; geometry collision mesh filename=package://berkeley_humanoid_lite_description/meshes_adapter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 scale=0.001 0.001 0.001; visual mesh filename=package://berkeley_humanoid_lite_description/meshes_adapter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 scale=0.001 0.001 0.001
- link arm_right_mount: mass None -> 0.0508; geometry collision mesh filename=package://berkeley_humanoid_lite_description/meshes_adapter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 scale=0.001 0.001 0.001; visual mesh filename=package://berkeley_humanoid_lite_description/meshes_adapter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 scale=0.001 0.001 0.001
Joints:
- joint arm_left_forearm_mount: origin xyz=0 -0 0 rpy=-0 0 -0 -> xyz=0 -0 0.012 rpy=-0 0 -0
- joint arm_right_forearm_mount: origin xyz=0 0 0 rpy=0 0 0 -> xyz=0 0 0.012 rpy=0 0 0

Commit message: Swap the forearm adapter for the lab's coupling part, and add an assembly STL exporter
The printed part between the elbow_roll flange and the V1 forearm is now the
lab's own SolidWorks part (cad/coupling_v2_2ea_original.STL as received; the
mesh in meshes_adapter/ is the same part moved into the elbow_roll frame).
It is a D72 x 8.5 mm disc on a D43 spigot that seats on the actuator output
ring like the stock hand did, bolts through the stock D36 pattern, and lives
in the D72 pocket inside the V1 forearm cuff. The forearm therefore moves
13.65 mm toward the elbow: mount z goes from +12 mm to -1.65 mm. Mass
properties are recomputed from the mesh at solid-PLA density. The design
notes and the open checks for the real arm are in arm_attachment.yaml.

scripts/merge_urdf_stl.py places every visual mesh of a URDF at a joint
pose and writes one STL (numpy only, resolves the Windows-broken mesh
symlinks itself). Its default output folder, export/, is ignored.

Co-Authored-By: Claude Opus 5.5 <noreply@anthropic.com>
Claude-Session: https://claude.ai/code/session_01HjX8F2k1kdozB2DdnpUNuM

File: ros2_ws/src/berkeley_humanoid_lite_description/urdf/berkeley_humanoid_lite_dexhand.urdf (robot description, URDF)
Before this commit: robot berkeley-humanoid-lite, 42 links, 41 joints
Links:
- link arm_right_mount: mass 0.0508 -> 0.0447
Joints:
- joint arm_right_forearm_mount: origin xyz=0 0 0.012 rpy=0 0 0 -> xyz=0 0 -0.00165 rpy=0 0 0

File: ros2_ws/src/berkeley_humanoid_lite_description/urdf/berkeley_humanoid_lite_tuning.urdf (robot description, URDF)
Before this commit: robot berkeley-humanoid-lite, 87 links, 86 joints
Links:
- link arm_left_mount: mass 0.0508 -> 0.0447
Joints:
- joint arm_left_forearm_mount: origin xyz=0 -0 0.012 rpy=-0 0 -0 -> xyz=0 -0 -0.00165 rpy=-0 0 -0

File: ros2_ws/src/berkeley_humanoid_lite_description/urdf/berkeley_humanoid_lite_v1arm.urdf (robot description, URDF)
Before this commit: robot berkeley-humanoid-lite, 82 links, 81 joints
Links:
- link arm_left_mount: mass 0.0508 -> 0.0447
- link arm_right_mount: mass 0.0508 -> 0.0447
Joints:
- joint arm_left_forearm_mount: origin xyz=0 -0 0.012 rpy=-0 0 -0 -> xyz=0 -0 -0.00165 rpy=-0 0 -0
- joint arm_right_forearm_mount: origin xyz=0 0 0.012 rpy=0 0 0 -> xyz=0 0 -0.00165 rpy=0 0 0
