Commit message: Mount the ZED 2i head on the torso, with a pan joint and the camera frames
The head is the lab's own part (cad/head_zed2i_mount_source.blend): a
printed bracket bolted with T-nuts to the inner face of the front top 2020
rail, a pan servo inside it, a lid, and a ZED 2i screwed onto the servo
horn. Its parts are exported from the blend into meshes_head/ (mm), with the
camera as a plain envelope of the ZED 2i's outside dimensions.

The placement is measured, not guessed, where the meshes allow it: the
bracket's wings are exactly the rail's 20 mm and their holes sit on the slot
centre (z 820 mm), and the rail's inner face is x 50 mm. Which face, and
left-right centring, are as built. The pan axis is the servo's output axis,
9.8 mm right of the centreline because the horn sits at one end of the body.

attach_head() in generate_urdf.py builds head_mount -> head_yaw (revolute)
-> head_pan -> the zed2i frames from Stereolabs' zed_macro.urdf.xacro, so
the wrapper's TF tree lines up, plus zed_imu_link where zed_imu_ros2
publishes. It is driven by the new `head` section of arm_attachment.yaml,
which also lists what is still unmeasured: servo model and mass, yaw
limits, the IMU's pose in the camera, and printed (not solid) part masses.
All four URDFs carry the head; the SRDFs are regenerated, which also adds
pairs for the coupling-v2 mount that the committed matrices predated.

merge_urdf_stl.py gains --subtree and --frame, used to write the head on
its own (export/head_zed2i_zero_pose_mm.stl) next to the full assembly.
tests/test_head.py pins the frames: on every model, forward at zero, left
camera on the left.

Co-Authored-By: Claude Opus 5.5 <noreply@anthropic.com>
Claude-Session: https://claude.ai/code/session_01HjX8F2k1kdozB2DdnpUNuM

File: ros2_ws/src/berkeley_humanoid_lite_description/urdf/berkeley_humanoid_lite.urdf (robot description, URDF)
Before this commit: robot berkeley-humanoid-lite, 16 links, 15 joints
Links:
- added link head_mount, mass 0.15045; collision mesh filename=package://berkeley_humanoid_lite_description/meshes_head/he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 scale=0.001 0.001 0.001; collision mesh filename=package://berkeley_humanoid_lite_description/meshes_head/he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 scale=0.001 0.001 0.001
- added link head_pan
- added link zed_camera_center, mass 0.166; collision mesh filename=package://berkeley_humanoid_lite_description/meshes_head/ze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 scale=0.001 0.001 0.001; visual mesh filename=package://berkeley_humanoid_lite_description/meshes_head/ze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 scale=0.001 0.001 0.001
- added link zed_camera_link
- added link zed_imu_link
- added link zed_left_camera_frame
- added link zed_left_camera_frame_optical
- added link zed_right_camera_frame
- added link zed_right_camera_frame_optical
Joints:
- added joint head_mount_joint: type fixed, parent base, child head_mount, origin xyz=0.05 0 0.82 rpy=0 0 3.14159265359
- added joint head_yaw: type revolute, parent head_mount, child head_pan, origin xyz=0.0247793 0.0098105 0.0289726 rpy=0 0 3.14159265359, axis 0 0 1, limit lower=-1.5708 upper=1.5708 effort=1.5 velocity=5.0
- added joint zed_camera_center_joint: type fixed, parent zed_camera_link, child zed_camera_center, origin xyz=0 0 0.015 rpy=0 0 0
- added joint zed_camera_joint: type fixed, parent head_pan, child zed_camera_link, origin xyz=0 0 0 rpy=0 0 0
- added joint zed_imu_joint: type fixed, parent zed_camera_center, child zed_imu_link, origin xyz=0 0 0 rpy=0 0 0
- added joint zed_left_camera_joint: type fixed, parent zed_camera_center, child zed_left_camera_frame, origin xyz=-0.01 0.06 0 rpy=0 0 0
- added joint zed_left_camera_optical_joint: type fixed, parent zed_left_camera_frame, child zed_left_camera_frame_optical, origin xyz=0 0 0 rpy=-1.57079632679 0 -1.57079632679
- added joint zed_right_camera_joint: type fixed, parent zed_camera_center, child zed_right_camera_frame, origin xyz=-0.01 -0.06 0 rpy=0 0 0
- added joint zed_right_camera_optical_joint: type fixed, parent zed_right_camera_frame, child zed_right_camera_frame_optical, origin xyz=0 0 0 rpy=-1.57079632679 0 -1.57079632679

File: ros2_ws/src/berkeley_humanoid_lite_description/urdf/berkeley_humanoid_lite_dexhand.urdf (robot description, URDF)
Before this commit: robot berkeley-humanoid-lite, 42 links, 41 joints
Links:
- added link head_mount, mass 0.15045; collision mesh filename=package://berkeley_humanoid_lite_description/meshes_head/he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 scale=0.001 0.001 0.001; collision mesh filename=package://berkeley_humanoid_lite_description/meshes_head/he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 scale=0.001 0.001 0.001
- added link head_pan
- added link zed_camera_center, mass 0.166; collision mesh filename=package://berkeley_humanoid_lite_description/meshes_head/ze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 scale=0.001 0.001 0.001; visual mesh filename=package://berkeley_humanoid_lite_description/meshes_head/ze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 scale=0.001 0.001 0.001
- added link zed_camera_link
- added link zed_imu_link
- added link zed_left_camera_frame
- added link zed_left_camera_frame_optical
- added link zed_right_camera_frame
- added link zed_right_camera_frame_optical
Joints:
- added joint head_mount_joint: type fixed, parent base, child head_mount, origin xyz=0.05 0 0.82 rpy=0 0 3.14159265359
- added joint head_yaw: type revolute, parent head_mount, child head_pan, origin xyz=0.0247793 0.0098105 0.0289726 rpy=0 0 3.14159265359, axis 0 0 1, limit lower=-1.5708 upper=1.5708 effort=1.5 velocity=5.0
- added joint zed_camera_center_joint: type fixed, parent zed_camera_link, child zed_camera_center, origin xyz=0 0 0.015 rpy=0 0 0
- added joint zed_camera_joint: type fixed, parent head_pan, child zed_camera_link, origin xyz=0 0 0 rpy=0 0 0
- added joint zed_imu_joint: type fixed, parent zed_camera_center, child zed_imu_link, origin xyz=0 0 0 rpy=0 0 0
- added joint zed_left_camera_joint: type fixed, parent zed_camera_center, child zed_left_camera_frame, origin xyz=-0.01 0.06 0 rpy=0 0 0
- added joint zed_left_camera_optical_joint: type fixed, parent zed_left_camera_frame, child zed_left_camera_frame_optical, origin xyz=0 0 0 rpy=-1.57079632679 0 -1.57079632679
- added joint zed_right_camera_joint: type fixed, parent zed_camera_center, child zed_right_camera_frame, origin xyz=-0.01 -0.06 0 rpy=0 0 0
- added joint zed_right_camera_optical_joint: type fixed, parent zed_right_camera_frame, child zed_right_camera_frame_optical, origin xyz=0 0 0 rpy=-1.57079632679 0 -1.57079632679

File: ros2_ws/src/berkeley_humanoid_lite_description/urdf/berkeley_humanoid_lite_tuning.urdf (robot description, URDF)
Before this commit: robot berkeley-humanoid-lite, 87 links, 86 joints
Links:
- added link head_mount, mass 0.15045; collision mesh filename=package://berkeley_humanoid_lite_description/meshes_head/he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 scale=0.001 0.001 0.001; collision mesh filename=package://berkeley_humanoid_lite_description/meshes_head/he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 scale=0.001 0.001 0.001
- added link head_pan
- added link zed_camera_center, mass 0.166; collision mesh filename=package://berkeley_humanoid_lite_description/meshes_head/ze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 scale=0.001 0.001 0.001; visual mesh filename=package://berkeley_humanoid_lite_description/meshes_head/ze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 scale=0.001 0.001 0.001
- added link zed_camera_link
- added link zed_imu_link
- added link zed_left_camera_frame
- added link zed_left_camera_frame_optical
- added link zed_right_camera_frame
- added link zed_right_camera_frame_optical
Joints:
- added joint head_mount_joint: type fixed, parent base, child head_mount, origin xyz=0.05 0 0.82 rpy=0 0 3.14159265359
- added joint head_yaw: type revolute, parent head_mount, child head_pan, origin xyz=0.0247793 0.0098105 0.0289726 rpy=0 0 3.14159265359, axis 0 0 1, limit lower=-1.5708 upper=1.5708 effort=1.5 velocity=5.0
- added joint zed_camera_center_joint: type fixed, parent zed_camera_link, child zed_camera_center, origin xyz=0 0 0.015 rpy=0 0 0
- added joint zed_camera_joint: type fixed, parent head_pan, child zed_camera_link, origin xyz=0 0 0 rpy=0 0 0
- added joint zed_imu_joint: type fixed, parent zed_camera_center, child zed_imu_link, origin xyz=0 0 0 rpy=0 0 0
- added joint zed_left_camera_joint: type fixed, parent zed_camera_center, child zed_left_camera_frame, origin xyz=-0.01 0.06 0 rpy=0 0 0
- added joint zed_left_camera_optical_joint: type fixed, parent zed_left_camera_frame, child zed_left_camera_frame_optical, origin xyz=0 0 0 rpy=-1.57079632679 0 -1.57079632679
- added joint zed_right_camera_joint: type fixed, parent zed_camera_center, child zed_right_camera_frame, origin xyz=-0.01 -0.06 0 rpy=0 0 0
- added joint zed_right_camera_optical_joint: type fixed, parent zed_right_camera_frame, child zed_right_camera_frame_optical, origin xyz=0 0 0 rpy=-1.57079632679 0 -1.57079632679

File: ros2_ws/src/berkeley_humanoid_lite_description/urdf/berkeley_humanoid_lite_v1arm.urdf (robot description, URDF)
Before this commit: robot berkeley-humanoid-lite, 82 links, 81 joints
Links:
- added link head_mount, mass 0.15045; collision mesh filename=package://berkeley_humanoid_lite_description/meshes_head/he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 scale=0.001 0.001 0.001; collision mesh filename=package://berkeley_humanoid_lite_description/meshes_head/he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 scale=0.001 0.001 0.001
- added link head_pan
- added link zed_camera_center, mass 0.166; collision mesh filename=package://berkeley_humanoid_lite_description/meshes_head/ze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 scale=0.001 0.001 0.001; visual mesh filename=package://berkeley_humanoid_lite_description/meshes_head/ze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 scale=0.001 0.001 0.001
- added link zed_camera_link
- added link zed_imu_link
- added link zed_left_camera_frame
- added link zed_left_camera_frame_optical
- added link zed_right_camera_frame
- added link zed_right_camera_frame_optical
Joints:
- added joint head_mount_joint: type fixed, parent base, child head_mount, origin xyz=0.05 0 0.82 rpy=0 0 3.14159265359
- added joint head_yaw: type revolute, parent head_mount, child head_pan, origin xyz=0.0247793 0.0098105 0.0289726 rpy=0 0 3.14159265359, axis 0 0 1, limit lower=-1.5708 upper=1.5708 effort=1.5 velocity=5.0
- added joint zed_camera_center_joint: type fixed, parent zed_camera_link, child zed_camera_center, origin xyz=0 0 0.015 rpy=0 0 0
- added joint zed_camera_joint: type fixed, parent head_pan, child zed_camera_link, origin xyz=0 0 0 rpy=0 0 0
- added joint zed_imu_joint: type fixed, parent zed_camera_center, child zed_imu_link, origin xyz=0 0 0 rpy=0 0 0
- added joint zed_left_camera_joint: type fixed, parent zed_camera_center, child zed_left_camera_frame, origin xyz=-0.01 0.06 0 rpy=0 0 0
- added joint zed_left_camera_optical_joint: type fixed, parent zed_left_camera_frame, child zed_left_camera_frame_optical, origin xyz=0 0 0 rpy=-1.57079632679 0 -1.57079632679
- added joint zed_right_camera_joint: type fixed, parent zed_camera_center, child zed_right_camera_frame, origin xyz=-0.01 -0.06 0 rpy=0 0 0
- added joint zed_right_camera_optical_joint: type fixed, parent zed_right_camera_frame, child zed_right_camera_frame_optical, origin xyz=0 0 0 rpy=-1.57079632679 0 -1.57079632679
